File: KiCadPCBFiles/HackPad.kicad_pcb (KiCad board)
At the start: 2 copper layers, 7 parts, among them SW1 SW_Push, SW2 SW_Push, SW3 SW_Push, SW4 SW_Push, SW5 SW_Push, SW6 SW_Push, U1 MOUDLE-SEEEDUINO-XIAO

Commit message: Add files via upload
Routing:
- net GND: track 0.00 -> 166.7 mm
Changed lines of the file:
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@@
+	)
+	(segment
+		(start 132.04 85)
+		(end 132.04 71.92)
+		(width 0.2)
+		(layer "B.Cu")
+		(net "GND")
+	)
+	(segment
+		(start 196.795 85)
+		(end 202.42 79.375)
+		(width 0.2)
+		(layer "B.Cu")
+		(net "GND")
+	)
+	(segment
+		(start 132.04 95.42)
+		(end 132.04 85)
+		(width 0.2)
+		(layer "B.Cu")
+		(net "GND")
+	)
+	(segment
+		(start 132.04 85)
+		(end 196.795 85)
+		(width 0.2)
+		(layer "B.Cu")
+		(net "GND")
+	)
+	(segment
+		(start 154.04 95.42)
+		(end 154.04 71.92)
+		(width 0.2)
+		(layer "B.Cu")
+		(net "GND")
+	)
+	(segment
+		(start 176.54 95.42)
+		(end 176.54 71.92)
+		(width 0.2)
+		(layer "B.Cu")
+		(net "GND")
+	)
+	(segment
+		(start 132.04 95.42)
+		(end 132.04 71.92)
+		(width 0.2)
+		(layer "B.Cu")
+		(net "GND")
 	)
 	(segment

Commit message: Add files via upload
Routing:
- net GND: track 166.7 -> 0.00 mm
Changed lines of the file:
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@@
-	)
-	(segment
-		(start 132.04 85)
-		(end 132.04 71.92)
-		(width 0.2)
-		(layer "B.Cu")
-		(net "GND")
-	)
-	(segment
-		(start 196.795 85)
-		(end 202.42 79.375)
-		(width 0.2)
-		(layer "B.Cu")
-		(net "GND")
-	)
-	(segment
-		(start 132.04 95.42)
-		(end 132.04 85)
-		(width 0.2)
-		(layer "B.Cu")
-		(net "GND")
-	)
-	(segment
-		(start 132.04 85)
-		(end 196.795 85)
-		(width 0.2)
-		(layer "B.Cu")
-		(net "GND")
-	)
-	(segment
-		(start 154.04 95.42)
-		(end 154.04 71.92)
-		(width 0.2)
-		(layer "B.Cu")
-		(net "GND")
-	)
-	(segment
-		(start 176.54 95.42)
-		(end 176.54 71.92)
-		(width 0.2)
-		(layer "B.Cu")
-		(net "GND")
-	)
-	(segment
-		(start 132.04 95.42)
-		(end 132.04 71.92)
-		(width 0.2)
-		(layer "B.Cu")
-		(net "GND")
 	)
 	(segment
@@
 		(min_thickness 0.25)
 		(fill yes
+			(mode hatch)
 			(thermal_gap 0.5)
 			(thermal_bridge_width 0.5)
 			(island_removal_mode 0)
+			(hatch_thickness 1)
+			(hatch_gap 1.5)
+			(hatch_orientation 0)
+			(hatch_border_algorithm hatch_thickness)
+			(hatch_min_hole_area 0.15)
 		)
 		(polygon
